File: pcb/zeta80-board/zeta80-board.kicad_sch (KiCad schematic)
At the start: 2 parts, among them IC1 SIO2-DIP-40, U1 Z80CPU

Commit message: Updating schematic
Parts:
- added C12, C13, C14, C15: 10uF, Capacitor_THT:CP_Radial_D5.0mm_P2.50mm, symbol Device:C_Polarized
- added C6, C7: 100nF, Capacitor_THT:C_Disc_D5.0mm_W2.5mm_P5.00mm, symbol Device:C
- added J2: UART1, Connector_Dsub:DSUB-9_Pins_Horizontal_P2.77x2.84mm_EdgePinOffset4.94mm_Housed_MountingHolesOffset4.94mm, symbol Connector:DE9_Pins_MountingHoles
- added R1, R2, R3: 2.7k, symbol Device:R
- added R10, R4, R6, R9: 10k, symbol Device:R
- added R5: 1k, symbol Device:R
- added R7, R8: 1k, Resistor_THT:R_Axial_DIN0207_L6.3mm_D2.5mm_P7.62mm_Horizontal, symbol Device:R
- added SW3, SW4: NMI, Button_Switch_THT:SW_PUSH_6mm, symbol Switch:SW_Push
- added U2: SST39SF010, symbol Memory_Flash:SST39SF010
- added U3: CY62256-70PC, Package_DIP:DIP-28_W15.24mm, symbol Memory_RAM:CY62256-70PC
- added U4: 74LS139, symbol 74xx:74LS139
- added U7: MAX232, Package_DIP:DIP-16_W7.62mm_Socket, symbol Interface_UART:MAX232
- added Y1: TCXO-14, Oscillator:Oscillator_DIP-14, symbol Oscillator:TCXO-14
Connections:
- net A0: now also IC1.34 (B/~{A}), U2.12 (A0), U3.10 (A0)
- net A1: now also IC1.33 (C/~{D}), U2.11 (A1), U3.9 (A1)
- net A10: now also U2.23 (A10), U3.21 (A10)
- net A11: now also U2.25 (A11), U3.23 (A11)
- net A12: now also U2.4 (A12), U3.2 (A12)
- net A13: now also U2.28 (A13), U3.26 (A13)
- net A14: now also U2.29 (A14), U3.1 (A14)
- net A15: now also U4.2 (A0)
- net A2: now also U2.10 (A2), U3.8 (A2)
- net A3: now also U2.9 (A3), U3.7 (A3)
- net A4: now also U2.8 (A4), U3.6 (A4), U4.14 (A0)
- net A5: now also U2.7 (A5), U3.5 (A5), U4.13 (A1)
- net A6: now also U2.6 (A6), U3.4 (A6)
- net A7: now also U2.5 (A7), U3.3 (A7)
- net A8: now also U2.27 (A8), U3.25 (A8)
- net A9: now also U2.26 (A9), U3.24 (A9)
- net CLK: now also IC1.20 (F), Y1.8 (OUT)
- net D0: now also IC1.40 (D0), U2.13 (D0), U3.11 (Q0)
- net D1: now also IC1.1 (D1), U2.14 (D1), U3.12 (Q1)
- net D2: now also IC1.39 (D2), U2.15 (D2), U3.13 (Q2)
- net D3: now also IC1.2 (D3), U2.17 (D3), U3.15 (Q3)
- net D4: now also IC1.38 (D4), U2.18 (D4), U3.16 (Q4)
- net D5: now also IC1.3 (D5), U2.19 (D5), U3.17 (Q5)
- net D6: now also IC1.37 (D6), U2.20 (D6), U3.18 (Q6)
- net D7: now also IC1.4 (D7), U2.21 (D7), U3.19 (Q7)
- net GND: now also IC1.18 (~{CTSA}), IC1.19 (~{DCDA}), C13.1, C6.2, C7.2, J2.5, SW3.1, SW4.1, U2.1 (NC), U2.16 (GND), U2.2 (A16), U2.3 (A15), U2.30 (NC), U3.14 (GND), U4.3 (A1), U4.8 (GND), U7.15 (GND), Y1.7 (GND)
- net VCC: now also C12.2, R10.2, R4.2, R5.1, R6.2, R7.2, R8.2, R9.2, U2.31 (PGM), U2.32 (VCC), U3.28 (VCC), U4.16 (VCC), U7.16 (VCC), Y1.14 (Vcc)
- net ~{INT}: now also IC1.5 (~{INT}), R9.1
- net ~{IORQ}: now also IC1.36 (~{IORQ}), U4.15 (E)
- net ~{M1}: now also IC1.8 (~{M1})
- net ~{MREQ}: now also U4.1 (E)
- net ~{RD}: now also IC1.32 (~{RD}), U2.24 (OE), U3.22 (~{OE})
- net ~{RES}: now also IC1.21 (~{RESET}), C7.1, R8.1, SW4.2
- net ~{WR}: now also U3.27 (~{WE})
- net at IC1.11 (~{SYNCA}): now also R4.1
- net at IC1.12 (RXDA): now also R1.1
- net SIO_CLK: now reaches IC1.13 (~{RXCA})
- net SIO_CLK: now also IC1.14 (~{TXCA})
- net at IC1.15 (TXDA): now also R2.1
- net at IC1.17 (~{RTSA}): now also R3.1
- net ~{SIO_CS}: now reaches IC1.35 (~{CE})
- net ~{SIO_CS}: now also U4.12 (O0)
- net at IC1.6 (IEI): now also R5.2
- net ~{NMI}: now reaches U1.17 (~{NMI})
- net ~{NMI}: now also C6.1, R7.1, SW3.2
- net at U1.24 (~{WAIT}): now also R10.1
- net at U1.25 (~{BUSRQ}): now also R6.1
- new net: C15.1, U7.1 (C1+)
- new net: J2.3, U7.13 (R1IN)
- new net: J2.2, U7.14 (T1OUT)
- new net: C12.1, U7.2 (VS+)
- new net: C15.2, U7.3 (C1-)
- new net: C14.1, U7.4 (C2+)
- new net: C14.2, U7.5 (C2-)
- new net: C13.2, U7.6 (VS-)
- new net: J2.8, U7.7 (T2OUT)
- new net RTS: R3.2, U7.10 (T2IN)
- new net RX: R1.2, U7.12 (R1OUT)
- new net TX: R2.2, U7.11 (T1IN)
- new net ~{RAM_CS}: U3.20 (~{CS}), U4.5 (O1)
- new net ~{ROM_CS}: U2.22 (CE), U4.4 (O0)
- no-connect marks 0 -> 28
Other:
- note added: "Signals are wired such that TxD <-> RxD ~{CTS} <-> ~{RTS} such that no null-modem cable is needed."
- moved on the sheet: IC1
